File: CDH.kicad_sch (KiCad schematic)
At the start: 36 parts, among them J1 PC104 H1, J2 PC104 H2, U1 STM32H745BITx

Commit message: added jtag, PAY connector, CANFD transceivers to schematic
Parts:
- added C26, C27, C28, C29: 100n, symbol Device:C
- added J3: G125-MH12605M4P, G125-MH12605M4P:HARWIN_G125-MH12605M4P, symbol G125-MH12605M4P:G125-MH12605M4P
- added J4: Conn_ARM_JTAG_SWD_10, symbol Connector:Conn_ARM_JTAG_SWD_10
- added JP2, JP3: SolderJumper_2_Open, symbol Jumper:SolderJumper_2_Open
- added R6, R7: 120, symbol Device:R
- added R8: 10K, symbol Device:R
- added U2, U3: MCP2562FDT-H_SN, MCP2562FDT-H_SN:SOIC127P600X175-8N, symbol MCP2562FDT-H_SN:MCP2562FDT-H_SN
Connections:
- net BAT is gone; now on net VDD: U1.8 (VBAT)
- net DEBUG_JTCK-SWCLK: now also J4.4 (SWCLK/TCK)
- net DEBUG_JTDI: now also J4.8 (NC/TDI)
- net DEBUG_JTDO-SWO: now also J4.6 (SWO/TDO)
- net DEBUG_JTMS-SWDIO: now also J4.2 (SWDIO/TMS)
- net FDCAN1_RX: now also U2.4 (RXD)
- net FDCAN1_TX: now also U2.1 (TXD)
- net FDCAN2_RX: now also U3.4 (RXD)
- net FDCAN2_TX: now also U3.1 (TXD)
- net GND: now also C26.1, C27.2, C28.1, C29.2, J3.14, J3.15, J3.16, J3.17, J3.18, J3.19, J4.3 (GND), J4.5 (GND), U2.2 (VSS), U2.8 (STBY), U3.2 (VSS), U3.8 (STBY)
- net I2C1_SCL: now also J3.20
- net I2C1_SDA: now also J3.21
- net PAY1: now also J3.25
- net PAY2: now also J3.24
- net PAY3: now also J3.23
- net PAY4: now also J3.22
- net SPI1_MISO: now also J3.6, J3.7
- net SPI1_SCK: now also J3.8
- net VDD: now also C26.2, C28.2, J3.4, J3.5, J4.1 (VTref), R8.1, U2.5 (VIO), U3.5 (VIO)
- net RESET: now reaches C25.1, SW_Reset.3 (K), SW_Reset.4 (A), U1.37 (NRST)
- net CS1: now reaches U1.143 (PC7)
- net CS1: now also J3.9
- net CS2: now reaches U1.144 (PC8)
- net CS2: now also J3.10
- net CS3: now reaches U1.145 (PC9)
- net CS3: now also J3.11
- net CS4: now reaches U1.146 (PA8)
- net CS4: now also J3.12
- net CS5: now reaches U1.147 (PA9)
- net CS5: now also J3.13
- net CS6: now reaches U1.148 (PA10)
- net CS6: now also J3.26
- net SPI2_MISO: no longer names the net of U1.40 (PC2_C)
- net SPI2_MOSI: no longer names the net of U1.39 (PC1)
- net SPI2_SCK: no longer names the net of U1.87 (PB10)
- new net: J4.10 (~{RESET}), R8.2
- new net: JP3.2 (B), R7.1
- new net: JP2.2 (B), R6.1
- new net +5V: C27.1, C29.1, J3.1, J3.2, J3.3, U2.3 (VDD), U3.3 (VDD)
- new net CANH_PC104: JP2.1 (A), JP3.1 (A), U2.7 (CANH), U3.7 (CANH)
- new net CANL_PC104: R6.2, R7.2, U2.6 (CANL), U3.6 (CANL)
- no-connect marks 2 -> 3

Commit message: done with schematic
Parts:
- removed C28, C29: 100n, symbol Device:C
- removed J1: PC104 H1, symbol Connector_Generic:Conn_02x26_Counter_Clockwise
- removed J2: PC104 H2, symbol Connector_Generic:Conn_02x26_Counter_Clockwise
- removed JP3: SolderJumper_2_Open, symbol Jumper:SolderJumper_2_Open
- removed R7: 120, symbol Device:R
- removed U3: MCP2562FDT-H_SN, MCP2562FDT-H_SN:SOIC127P600X175-8N, symbol MCP2562FDT-H_SN:MCP2562FDT-H_SN
- added PC104_H1, PC104_H2: Conn_02x26_Odd_Even, symbol Connector_Generic:Conn_02x26_Odd_Even
Connections:
- net +5V: now also PC104_H2.25 (Pin_25), PC104_H2.26 (Pin_26)
- net CANH_PC104: now also PC104_H1.3 (Pin_3)
- net CANL_PC104: now also PC104_H1.1 (Pin_1)
- net GND: now also PC104_H2.29 (Pin_29), PC104_H2.30 (Pin_30)
- net I2C2_SCL: now also PC104_H1.43 (Pin_43)
- net I2C2_SDA: now also PC104_H1.41 (Pin_41)
- net VDD: now also PC104_H2.27 (Pin_27), PC104_H2.28 (Pin_28)
- net FDCAN2_RX: no longer names the net of U1.88 (PB11)
- net FDCAN2_TX: no longer names the net of U1.101 (PB12)
